Commit message: rotate UR5 base -pi/2 to make it correspond to our husky installation

File: mt_husky_moveit_config/urdf/husky_ur5_e.urdf (robot description, URDF)
Before this commit: robot husky, 28 links, 27 joints
Joints:
- joint ur_arm_base_link-base_fixed_joint: origin xyz=0 0 0 rpy=0 0 3.14159265359 -> xyz=0 0 0 rpy=0 0 -1.570796326795
- joint ur_arm_base_link-base_link_inertia: origin xyz=0 0 0 rpy=0 0 3.14159265359 -> xyz=0 0 0 rpy=0 0 -1.570796326795

Commit message: add bar tcp

File: mt_husky_moveit_config/urdf/husky_ur5_e.urdf (robot description, URDF)
Before this commit: robot husky, 28 links, 27 joints
Links:
- added link bar_tcp
- added link robotiq_85_mount
Joints:
- added joint mount_on_flange: type fixed, parent ur_arm_tool0, child robotiq_85_mount, origin xyz=0.0 0.0 0.0 rpy=0.0 0.0 0.0
- added joint tool0-bar_tcp_fixed_joint: type fixed, parent robotiq_85_mount, child bar_tcp, origin xyz=0 0 0.138 rpy=0 0 3.141592653589793

Commit message: add ipad rack

File: mt_husky_moveit_config/urdf/husky_ur5_e.urdf (robot description, URDF)
Before this commit: robot husky, 30 links, 29 joints
Links:
- added link ipad_rack_link; collision mesh filename=package://husky_description/meshes/ipad_rack_collision.obj; visual mesh filename=package://husky_description/meshes/ipad_rack_visual.obj
Joints:
- added joint ipad_rack_joint: type fixed, parent base_link, child ipad_rack_link, origin xyz=0.0812 0 0.225 rpy=0 0 0

Commit message: Update grasp for Victor's finger tip design

File: mt_husky_moveit_config/urdf/husky_ur5_e.urdf (robot description, URDF)
Before this commit: robot husky, 31 links, 30 joints
Joints:
- joint tool0-bar_tcp_fixed_joint: origin xyz=0 0 0.138 rpy=0 0 3.141592653589793 -> xyz=0 0 0.152 rpy=0 0 3.141592653589793

File: mt_husky_moveit_config/urdf/husky_ur5_e_no_base_joint.urdf (robot description, URDF)
Before this commit: robot husky, 29 links, 28 joints
Joints:
- joint tool0-bar_tcp_fixed_joint: origin xyz=0 0 0.138 rpy=0 0 3.141592653589793 -> xyz=0 0 0.152 rpy=0 0 3.141592653589793
