Commit message: comment out grasp to avoid confusion

File: mt_husky_moveit_config/urdf/husky_ur5_e_no_base_joint.urdf (robot description, URDF)
Before this commit: robot husky, 29 links, 28 joints
Links:
- removed link bar_tcp
Joints:
- removed joint tool0-bar_tcp_fixed_joint

Commit message: use relative path instead of  package://

File: mt_husky_moveit_config/urdf/husky_ur5_e_no_base_joint.urdf (robot description, URDF)
Before this commit: robot husky, 28 links, 27 joints
Links:
- link base_link: geometry collision box size=0.78992 0.5709 0.10375; visual mesh filename=../../husky_description/meshes/base_link.stl
- link front_bumper_link: geometry visual mesh filename=../../husky_description/meshes/bumper.obj
- link front_left_wheel_link: geometry collision cylinder length=0.1143 radius=0.1651; visual mesh filename=../../husky_description/meshes/wheel.obj
- link front_right_wheel_link: geometry collision cylinder length=0.1143 radius=0.1651; visual mesh filename=../../husky_description/meshes/wheel.obj
- link ipad_rack_link: geometry collision mesh filename=../../husky_description/meshes/ipad_rack_collision.obj; visual mesh filename=../../husky_description/meshes/ipad_rack_visual.obj
- link rear_bumper_link: geometry visual mesh filename=../../husky_description/meshes/bumper.obj
- link rear_left_wheel_link: geometry collision cylinder length=0.1143 radius=0.1651; visual mesh filename=../../husky_description/meshes/wheel.obj
- link rear_right_wheel_link: geometry collision cylinder length=0.1143 radius=0.1651; visual mesh filename=../../husky_description/meshes/wheel.obj
- link top_chassis_link: geometry visual mesh filename=../../husky_description/meshes/top_chassis.obj
- link top_plate_link: geometry collision mesh filename=../../husky_description/meshes/large_top_plate_collision.stl; visual mesh filename=../../husky_description/meshes/large_top_plate.obj
- link ur_arm_base_link_inertia: geometry collision mesh filename=../../ur_description/meshes/ur5e/collision/base.stl; visual mesh filename=../../ur_description/meshes/ur5e/visual/base.obj
- link ur_arm_forearm_link: geometry collision mesh filename=../../ur_description/meshes/ur5e/collision/forearm.stl; visual mesh filename=../../ur_description/meshes/ur5e/visual/forearm.obj
- link ur_arm_shoulder_link: geometry collision mesh filename=../../ur_description/meshes/ur5e/collision/shoulder.stl; visual mesh filename=../../ur_description/meshes/ur5e/visual/shoulder.obj
- link ur_arm_upper_arm_link: geometry collision mesh filename=../../ur_description/meshes/ur5e/collision/upperarm.stl; visual mesh filename=../../ur_description/meshes/ur5e/visual/upperarm.obj
- link ur_arm_wrist_1_link: geometry collision mesh filename=../../ur_description/meshes/ur5e/collision/wrist1.stl; visual mesh filename=../../ur_description/meshes/ur5e/visual/wrist1.obj
- link ur_arm_wrist_2_link: geometry collision mesh filename=../../ur_description/meshes/ur5e/collision/wrist2.stl; visual mesh filename=../../ur_description/meshes/ur5e/visual/wrist2.obj
- link ur_arm_wrist_3_link: geometry collision mesh filename=../../ur_description/meshes/ur5e/collision/wrist3.stl; visual mesh filename=../../ur_description/meshes/ur5e/visual/wrist3.obj
