Commit message: cindy urdf cleanup wip - base done

File: mt_husky_dual_ur5_e_moveit_config/urdf/temp.urdf (robot description, URDF)
Before this commit: robot husky, 36 links, 35 joints
Links:
- removed link base_footprint
- removed link base_link
- removed link front_left_wheel_link
- removed link imu_link
- removed link inertial_link
Joints:
- removed joint base_footprint_joint
- removed joint front_left_wheel
- removed joint imu_joint
- removed joint inertial_joint
