Commit message: Cleanup dual-arm husky udrf - a lot of duplicated sections messed up compas loading

File: mt_husky_dual_ur5_e_moveit_config/urdf/husky_dual_ur5_e.urdf (robot description, URDF)
Before this commit: robot husky, 36 links, 35 joints
Links:
- added link base_link_0
- added link base_link_1
- added link world_link
- link base_link: geometry collision box size=0.78992 0.5709 0.10375; collision box size=0.9874 0.5709 0.12375
Joints:
- added joint theta: type continuous, parent base_link_1, child base_footprint, axis 0 0 1, limit effort=1000.0 velocity=1.5708
- added joint x: type prismatic, parent world_link, child base_link_0, axis 1 0 0, limit lower=-5 upper=5 effort=1000.0 velocity=1.0
- added joint y: type prismatic, parent base_link_0, child base_link_1, axis 0 1 0, limit lower=-5 upper=5 effort=1000.0 velocity=1.0

File: mt_husky_dual_ur5_e_moveit_config/urdf/husky_dual_ur5_e_no_base_joint.urdf (robot description, URDF)
Before this commit: robot husky, 31 links, 31 joints
Links:
- added link base_footprint
- added link base_link, mass 0.1; collision box size=0.78992 0.5709 0.10375; collision box size=0.9874 0.5709 0.12375
- added link front_left_wheel_link, mass 2.637; collision cylinder length=0.1143 radius=0.1651; visual mesh filename=package://husky_description/meshes/wheel.obj
- added link imu_link
- added link inertial_link, mass 46.034
Joints:
- added joint base_footprint_joint: type fixed, parent base_link, child base_footprint, origin xyz=0 0 -0.13228 rpy=0 0 0
- added joint front_left_wheel: type continuous, parent base_link, child front_left_wheel_link, origin xyz=0.256 0.2854 0.03282 rpy=0 0 0, axis 0 1 0
- added joint imu_joint: type fixed, parent base_link, child imu_link, origin xyz=0.19 0 0.149 rpy=0 -1.5708 3.1416
- added joint inertial_joint: type fixed, parent base_link, child inertial_link, origin xyz=0 0 0 rpy=0 0 0

Commit message: fix wheeled joint - still can't get the base xytheta joints work but that's for later

File: mt_husky_dual_ur5_e_moveit_config/urdf/husky_dual_ur5_e.urdf (robot description, URDF)
Before this commit: robot husky, 39 links, 38 joints
Joints:
- joint front_left_wheel: type continuous -> fixed
- joint front_right_wheel: type continuous -> fixed
- joint rear_left_wheel: type continuous -> fixed
- joint rear_right_wheel: type continuous -> fixed

File: mt_husky_moveit_config/urdf/husky_ur5_e.urdf (robot description, URDF)
Before this commit: robot husky, 31 links, 30 joints
Joints:
- joint front_left_wheel: type continuous -> fixed
- joint front_right_wheel: type continuous -> fixed
- joint rear_left_wheel: type continuous -> fixed
- joint rear_right_wheel: type continuous -> fixed

Commit message: fix flipped base_link and footprint link bug in dual arm

File: mt_husky_dual_ur5_e_moveit_config/urdf/husky_dual_ur5_e.urdf (robot description, URDF)
Before this commit: robot husky, 39 links, 38 joints
Joints:
- joint base_footprint_joint: child base_footprint -> base_link; parent base_link -> base_footprint
