Commit message: fix footprint link in Cindy no basejoint

File: mt_husky_dual_ur5_e_moveit_config/urdf/husky_dual_ur5_e_no_base_joint.urdf (robot description, URDF)
Before this commit: robot husky, 36 links, 35 joints
Links:
- added link world_link
Joints:
- added joint world_footprint: type fixed, parent world_link, child base_footprint, origin xyz=0 0 0 rpy=0 0 0
- joint base_footprint_joint: child base_footprint -> base_link; parent base_link -> base_footprint

Commit message: fix incorrect footprint joint offset

File: mt_husky_dual_ur5_e_moveit_config/urdf/husky_dual_ur5_e_no_base_joint.urdf (robot description, URDF)
Before this commit: robot husky, 37 links, 36 joints
Joints:
- joint base_footprint_joint: origin xyz=0 0 -0.13228 rpy=0 0 0 -> xyz=0 0 0.13228 rpy=0 0 0
- joint right_ur_arm_base_link-base_fixed_joint: origin xyz=0 0 0 rpy=0 0 3.14159265359 -> xyz=0 0 0 rpy=0 0 -1.570796326795

Commit message: comment out all gazebo and transmission stuff in the husky urdfs

File: mt_husky_dual_ur5_e_moveit_config/urdf/husky_dual_ur5_e_no_base_joint.urdf (robot description, URDF)
Before this commit: robot husky, 37 links, 36 joints
Joints:
- joint front_left_wheel: type continuous -> fixed
- joint front_right_wheel: type continuous -> fixed
- joint rear_left_wheel: type continuous -> fixed
- joint rear_right_wheel: origin xyz=-0.256 -0.2854 0.03282 rpy=0 0 0 -> xyz=-0.48 0 0.091 rpy=0 0 3.14159; type continuous -> fixed
- joint right_ur_arm_base_link-base_link_inertia: origin xyz=0 0 0 rpy=0 0 3.14159265359 -> xyz=0 0 0 rpy=0 0 -1.570796326795

File: mt_husky_moveit_config/urdf/husky_ur5_e_no_base_joint.urdf (robot description, URDF)
Before this commit: robot husky, 28 links, 27 joints
Joints:
- joint front_left_wheel: type continuous -> fixed
- joint front_right_wheel: type continuous -> fixed
- joint rear_left_wheel: type continuous -> fixed
- joint rear_right_wheel: type continuous -> fixed

Commit message: Fix some rand joint change from Cursor

File: mt_husky_dual_ur5_e_moveit_config/urdf/husky_dual_ur5_e_no_base_joint.urdf (robot description, URDF)
Before this commit: robot husky, 37 links, 36 joints
Joints:
- joint rear_right_wheel: origin xyz=-0.48 0 0.091 rpy=0 0 3.14159 -> xyz=-0.256 -0.2854 0.03282 rpy=0 0 0
- joint right_ur_arm_base_link-base_link_inertia: origin xyz=0 0 0 rpy=0 0 -1.570796326795 -> xyz=0 0 0 rpy=0 0 3.14159265359

Commit message: Limits joint ranges for the UR5 arms
Reduces the joint limits for the shoulder and shoulder lift joints on both UR5 arms.

This change prevents the robot from exceeding its physical limitations and potentially causing damage to itself or its surroundings.
The limits are adjusted to ensure safe operation within the workspace.

File: mt_husky_dual_ur5_e_moveit_config/urdf/husky_dual_ur5_e_no_base_joint.urdf (robot description, URDF)
Before this commit: robot husky, 37 links, 36 joints
Joints:
- joint left_ur_arm_shoulder_lift_joint: limit lower=-6.28318530718 upper=6.28318530718 effort=150.0 velocity=3.14159265359 -> lower=-3.14159265359 upper=0.3 effort=150.0 velocity=3.14159265359
- joint left_ur_arm_shoulder_pan_joint: limit lower=-6.28318530718 upper=6.28318530718 effort=150.0 velocity=3.14159265359 -> lower=-3.14159265359 upper=3.14159265359 effort=150.0 velocity=3.14159265359
- joint right_ur_arm_shoulder_lift_joint: limit lower=-6.28318530718 upper=6.28318530718 effort=150.0 velocity=3.14159265359 -> lower=-3.14159265359 upper=0.3 effort=150.0 velocity=3.14159265359
- joint right_ur_arm_shoulder_pan_joint: limit lower=-6.28318530718 upper=6.28318530718 effort=150.0 velocity=3.14159265359 -> lower=-3.14159265359 upper=3.14159265359 effort=150.0 velocity=3.14159265359

Commit message: Limits UR wrist joint range for Cindy
Reduces the range of motion for the UR wrist joints
to +/- pi to prevent joint limit errors and improve
robot behavior.

File: mt_husky_dual_ur5_e_moveit_config/urdf/husky_dual_ur5_e_no_base_joint.urdf (robot description, URDF)
Before this commit: robot husky, 37 links, 36 joints
Joints:
- joint left_ur_arm_wrist_1_joint: limit lower=-6.28318530718 upper=6.28318530718 effort=28.0 velocity=3.14159265359 -> lower=-4.18879020479 upper=4.18879020479 effort=28.0 velocity=3.14159265359
- joint left_ur_arm_wrist_2_joint: limit lower=-6.28318530718 upper=6.28318530718 effort=28.0 velocity=3.14159265359 -> lower=-4.18879020479 upper=4.18879020479 effort=28.0 velocity=3.14159265359
- joint left_ur_arm_wrist_3_joint: limit lower=-6.28318530718 upper=6.28318530718 effort=28.0 velocity=3.14159265359 -> lower=-4.18879020479 upper=4.18879020479 effort=28.0 velocity=3.14159265359
- joint right_ur_arm_wrist_1_joint: limit lower=-6.28318530718 upper=6.28318530718 effort=28.0 velocity=3.14159265359 -> lower=-4.18879020479 upper=4.18879020479 effort=28.0 velocity=3.14159265359
- joint right_ur_arm_wrist_2_joint: limit lower=-6.28318530718 upper=6.28318530718 effort=28.0 velocity=3.14159265359 -> lower=-4.18879020479 upper=4.18879020479 effort=28.0 velocity=3.14159265359
- joint right_ur_arm_wrist_3_joint: limit lower=-6.28318530718 upper=6.28318530718 effort=28.0 velocity=3.14159265359 -> lower=-4.18879020479 upper=4.18879020479 effort=28.0 velocity=3.14159265359
