Commit message: Calibrates UR5e arm poses
Updates joint origins in the URDF to calibrated values for both UR5e arms, improving pose accuracy.
This commit addresses inaccuracies in the robot's kinematic model using values got from hardware.

File: mt_husky_dual_ur5_e_moveit_config/urdf/husky_dual_ur5_e_no_base_joint_Calibrated.urdf (robot description, URDF)
Before this commit: robot husky, 37 links, 36 joints
Joints:
- joint left_ur_arm_elbow_joint: origin xyz=-0.425 0 0 rpy=0 0 0 -> xyz=-0.42492076346025309 0 0 rpy=0.00053885028029254363 -0.00088899660595502864 -0.0000090893692096143134
- joint left_ur_arm_shoulder_lift_joint: origin xyz=0 0 0 rpy=1.570796327 0 0 -> xyz=0.00019007197441139241 0 0 rpy=1.5713901981958054 0 -0.0000026681008682416518
- joint left_ur_arm_shoulder_pan_joint: origin xyz=0 0 0.1625 rpy=0 0 0 -> xyz=0 0 0.16257807277263761 rpy=0 0 0
- joint left_ur_arm_wrist_1_joint: origin xyz=-0.3922 0 0.1333 rpy=0 0 0 -> xyz=-0.39208100648997279 -0.00090760192761138176 0.13352893003432456 rpy=0.0067969386915389153 0.0021092387583197063 -0.0000069072557868343565
- joint left_ur_arm_wrist_2_joint: origin xyz=0 -0.0997 -2.0448811823e-11 rpy=1.570796327 0 0 -> xyz=0.00013627350480989177 -0.099746834502379381 0.0000073743752427287777 rpy=1.5707223958750225 0 -0.00000021941801741677536
- joint left_ur_arm_wrist_3_joint: origin xyz=0 0.0996 -2.04283014801e-11 rpy=1.57079632659 3.14159265359 3.14159265359 -> xyz=0.000025819376543512202 0.099466410942852038 0.000018368979052949448 rpy=1.5709810019899699 3.1415926535897931 -3.1415925563992939
- joint right_ur_arm_elbow_joint: origin xyz=-0.425 0 0 rpy=0 0 0 -> xyz=-0.42484922240722683 0 0 rpy=0.000017598778356909152 -0.0017646390504777454 0.000022896679262627857
- joint right_ur_arm_shoulder_lift_joint: origin xyz=0 0 0 rpy=1.570796327 0 0 -> xyz=0.00017951387097150235 0 0 rpy=1.5703872163784984 0 -0.0000044300287598275637
- joint right_ur_arm_shoulder_pan_joint: origin xyz=0 0 0.1625 rpy=0 0 0 -> xyz=0 0 0.1627782525221701 rpy=0 0 0
- joint right_ur_arm_wrist_1_joint: origin xyz=-0.3922 0 0.1333 rpy=0 0 0 -> xyz=-0.39267466285441494 -0.0007932258609161224 0.13276574606781064 rpy=0.0059745562860579046 -0.0017403184893875676 -0.000012182431672809177
- joint right_ur_arm_wrist_2_joint: origin xyz=0 -0.0997 -2.0448811823e-11 rpy=1.570796327 0 0 -> xyz=-0.000057633117397977084 -0.099557455213209314 0.00015287024635024139 rpy=1.569260830273018 0 0.00000037474165375667162
- joint right_ur_arm_wrist_3_joint: origin xyz=0 0.0996 -2.04283014801e-11 rpy=1.57079632659 3.14159265359 3.14159265359 -> xyz=0.000058942281949617339 0.099514048224567206 0.00020241494029680382 rpy=1.5728303578162324 3.1415926535897931 3.1415917754729397
