Commit message: Calibrates Cindy right arm mount joint transform
Corrects the transform of the right arm mount joint to improve the robot's accuracy.
This involves adjusting the rotation and translation values for a more precise alignment.

File: mt_husky_dual_ur5_e_moveit_config/urdf/husky_dual_ur5_e_no_base_joint_All_Calibrated.urdf (robot description, URDF)
Before this commit: robot husky, 37 links, 36 joints
Joints:
- joint right_arm_mount_joint: origin xyz=0 0 0 rpy=0 0 0 -> xyz=0.0011497288942337036 -0.0006287879659794271 0.002082839608192444 rpy=0.005849556200320057 -0.004160215708736291 -0.0035193052610289406

Commit message: enlarge joint limit

File: mt_husky_dual_ur5_e_moveit_config/urdf/husky_dual_ur5_e_no_base_joint_All_Calibrated.urdf (robot description, URDF)
Before this commit: robot husky, 37 links, 36 joints
Joints:
- joint left_ur_arm_shoulder_lift_joint: limit lower=-3.14159265359 upper=0.3 effort=150.0 velocity=3.14159265359 -> lower=-4.71238898038 upper=4.71238898038 effort=150.0 velocity=3.14159265359
- joint left_ur_arm_shoulder_pan_joint: limit lower=-3.14159265359 upper=3.14159265359 effort=150.0 velocity=3.14159265359 -> lower=-4.71238898038 upper=4.71238898038 effort=150.0 velocity=3.14159265359
- joint right_ur_arm_shoulder_lift_joint: limit lower=-3.14159265359 upper=0.3 effort=150.0 velocity=3.14159265359 -> lower=-4.71238898038 upper=4.71238898038 effort=150.0 velocity=3.14159265359
- joint right_ur_arm_shoulder_pan_joint: limit lower=-3.14159265359 upper=3.14159265359 effort=150.0 velocity=3.14159265359 -> lower=-4.71238898038 upper=4.71238898038 effort=150.0 velocity=3.14159265359

Commit message: enlarge Cindy's both arms' shoulder pan joint to avoid always in out of limit config after manual jog

File: mt_husky_dual_ur5_e_moveit_config/urdf/husky_dual_ur5_e_no_base_joint_All_Calibrated.urdf (robot description, URDF)
Before this commit: robot husky, 37 links, 36 joints
Joints:
- joint left_ur_arm_shoulder_pan_joint: limit lower=-4.71238898038 upper=4.71238898038 effort=150.0 velocity=3.14159265359 -> lower=-6.28318530718 upper=6.28318530718 effort=150.0 velocity=3.14159265359
- joint right_ur_arm_shoulder_pan_joint: limit lower=-4.71238898038 upper=4.71238898038 effort=150.0 velocity=3.14159265359 -> lower=-6.28318530718 upper=6.28318530718 effort=150.0 velocity=3.14159265359
