Commit message: ur base frames fixed in place, stock-frame copies removed
The fixed joints below each arm's base_link are back at the stock UR 180 degrees, and the arm's mounting turn is in
the mount joint above it. Comments next to both say which change goes where.

Co-Authored-By: Claude Opus 5.5 <noreply@anthropic.com>

File: husky_dual_ur5e_vamp.urdf (robot description, URDF)
Before this commit: robot dual-arm_husky_Cindy, 37 links, 36 joints
Joints:
- joint right_ur_arm_base_link-base_fixed_joint: origin xyz=0 0 0 rpy=0 0 -1.570796326795 -> xyz=0 0 0 rpy=0 0 3.14159265359

File: husky_ur_description/urdf/husky_ur5_e_description.urdf.xacro (robot description, xacro)
@@ -5,5 +5,7 @@
     <parent link="top_plate_front_link" />
     <child link="ur_arm_base_link" />
-    <origin xyz="$(optenv HUSKY_UR_XYZ -0.105 0.0 0.0)" rpy="$(optenv HUSKY_UR_RPY 0 0 3.1415927)"/>
+    <!-- The arm sits turned 90 deg on the top plate; that turn belongs here, never in the joints below
+         ur_arm_base_link (stock rpy 0 0 pi in ur_macro.xacro). -->
+    <origin xyz="$(optenv HUSKY_UR_XYZ -0.105 0.0 0.0)" rpy="$(optenv HUSKY_UR_RPY 0 0 -1.5707963)"/>
   </joint>
   <xacro:ur5e_robot prefix="ur_arm_" />

File: mt_husky_dual_ur5_e_moveit_config/urdf/husky_dual_ur5_e_no_base_joint.urdf (robot description, URDF)
Before this commit: robot husky, 37 links, 36 joints
Joints:
- joint right_ur_arm_base_link-base_fixed_joint: origin xyz=0 0 0 rpy=0 0 -1.570796326795 -> xyz=0 0 0 rpy=0 0 3.14159265359

File: mt_husky_dual_ur5_e_moveit_config/urdf/husky_dual_ur5_e_no_base_joint_All_Calibrated_objs.urdf (robot description, URDF)
Before this commit: robot husky, 37 links, 36 joints
Joints:
- joint right_ur_arm_base_link-base_fixed_joint: origin xyz=0 0 0 rpy=0 0 -1.570796326795 -> xyz=0 0 0 rpy=0 0 3.14159265359

File: mt_husky_dual_ur5_e_moveit_config/urdf/husky_dual_ur5_e_no_base_joint_Arm_Calibrated.urdf (robot description, URDF)
Before this commit: robot husky, 37 links, 36 joints
Joints:
- joint right_ur_arm_base_link-base_fixed_joint: origin xyz=0 0 0 rpy=0 0 -1.570796326795 -> xyz=0 0 0 rpy=0 0 3.14159265359

File: mt_husky_moveit_config/urdf/husky_ur5_e_no_base_joint.urdf (robot description, URDF)
Before this commit: robot husky, 28 links, 27 joints
Joints:
- joint arm_mount_joint: origin xyz=-0.105 0.0 0.0 rpy=0 0 3.1415927 -> xyz=-0.105 0.0 0.0 rpy=0 0 -1.57079628038
- joint ur_arm_base_link-base_fixed_joint: origin xyz=0 0 0 rpy=0 0 -1.570796326795 -> xyz=0 0 0 rpy=0 0 3.14159265359
- joint ur_arm_base_link-base_link_inertia: origin xyz=0 0 0 rpy=0 0 -1.570796326795 -> xyz=0 0 0 rpy=0 0 3.14159265359

File: mt_husky_moveit_config/urdf/husky_ur5_e_no_base_joint_Alice_Calibrated.urdf (robot description, URDF)
Before this commit: robot single-arm_husky_Alice, 28 links, 27 joints
Joints:
- joint arm_mount_joint: origin xyz=-0.105 0.0 0.0 rpy=0 0 3.1415927 -> xyz=-0.105 0.0 0.0 rpy=0 0 -1.57079628038
- joint ur_arm_base_link-base_fixed_joint: origin xyz=0 0 0 rpy=0 0 -1.570796326795 -> xyz=0 0 0 rpy=0 0 3.14159265359
- joint ur_arm_base_link-base_link_inertia: origin xyz=0 0 0 rpy=0 0 -1.570796326795 -> xyz=0 0 0 rpy=0 0 3.14159265359

File: mt_husky_moveit_config/urdf/husky_ur5_e_no_base_joint_Belle_Calibrated.urdf (robot description, URDF)
Before this commit: robot single-arm_husky_Belle, 28 links, 27 joints
Joints:
- joint arm_mount_joint: origin xyz=-0.105 0.0 0.0 rpy=0 0 3.1415927 -> xyz=-0.105 0.0 0.0 rpy=0 0 -1.57079628038
- joint ur_arm_base_link-base_fixed_joint: origin xyz=0 0 0 rpy=0 0 -1.570796326795 -> xyz=0 0 0 rpy=0 0 3.14159265359
- joint ur_arm_base_link-base_link_inertia: origin xyz=0 0 0 rpy=0 0 -1.570796326795 -> xyz=0 0 0 rpy=0 0 3.14159265359

Commit message: ipad rack boxes, cindy's ipad and single-arm floor box in the collision shapes
Calibration paths collided with the oversized iPad rack box, which prompted a check of every collision shape. The rack
is now boxes around its parts with a 1 cm margin, Cindy's bulkhead gets a box for her iPad, and Alice and Belle get
the floor box over their bumpers.

Co-Authored-By: Claude Opus 5.5 <noreply@anthropic.com>

File: husky_dual_ur5e_vamp.urdf (robot description, URDF)
Before this commit: robot dual-arm_husky_Cindy, 37 links, 36 joints
Links:
- link dual_arm_bulkhead_link: geometry collision box size=0.21 0.29 0.06; collision mesh filename=package://husky_ur_description/meshes/dual_arm_bulkhead_col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

File: mt_husky_dual_ur5_e_moveit_config/urdf/husky_dual_ur5_e_no_base_joint.urdf (robot description, URDF)
Before this commit: robot husky, 37 links, 36 joints
Links:
- link dual_arm_bulkhead_link: geometry collision box size=0.21 0.29 0.06; collision mesh filename=package://husky_ur_description/meshes/dual_arm_bulkhead_col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

File: mt_husky_dual_ur5_e_moveit_config/urdf/husky_dual_ur5_e_no_base_joint_Arm_Calibrated.urdf (robot description, URDF)
Before this commit: robot husky, 37 links, 36 joints
Links:
- link dual_arm_bulkhead_link: geometry collision box size=0.21 0.29 0.06; collision mesh filename=package://husky_ur_description/meshes/dual_arm_bulkhead_col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

File: mt_husky_moveit_config/urdf/husky_ur5_e_no_base_joint.urdf (robot description, URDF)
Before this commit: robot husky, 28 links, 27 joints
Links:
- link base_link: geometry collision box size=0.78992 0.5709 0.10375; collision box size=0.9874 0.5709 0.12375
- link ipad_rack_link: geometry collision box size=0.05 0.09 0.17; collision box size=0.06 0.5475 0.53

File: mt_husky_moveit_config/urdf/husky_ur5_e_no_base_joint_Alice_Calibrated.urdf (robot description, URDF)
Before this commit: robot single-arm_husky_Alice, 28 links, 27 joints
Links:
- link base_link: geometry collision box size=0.78992 0.5709 0.10375; collision box size=0.9874 0.5709 0.12375
- link ipad_rack_link: geometry collision box size=0.05 0.09 0.17; collision box size=0.06 0.5475 0.53

File: mt_husky_moveit_config/urdf/husky_ur5_e_no_base_joint_Belle_Calibrated.urdf (robot description, URDF)
Before this commit: robot single-arm_husky_Belle, 28 links, 27 joints
Links:
- link base_link: geometry collision box size=0.78992 0.5709 0.10375; collision box size=0.9874 0.5709 0.12375
- link ipad_rack_link: geometry collision box size=0.05 0.09 0.17; collision box size=0.06 0.5475 0.53
